Commit message: obstacle detected

File: src/mower_robot/urdf/mower_robot.urdf (robot description, URDF)
Before this commit: robot mower_robot, 5 links, 4 joints
Links:
- removed link caster_wheel
- removed link left_wheel
- removed link right_wheel
- added link left_front_caster, mass 0.5; collision cylinder length=0.05 radius=0.1; visual cylinder length=0.05 radius=0.1
- added link left_rear_wheel, mass 0.5; collision cylinder length=0.05 radius=0.1; visual cylinder length=0.05 radius=0.1
- added link right_front_caster, mass 0.5; collision cylinder length=0.05 radius=0.1; visual cylinder length=0.05 radius=0.1
- added link right_rear_wheel, mass 0.5; collision cylinder length=0.05 radius=0.1; visual cylinder length=0.05 radius=0.1
- link base_link: geometry collision box size=0.4 0.3 0.1; visual box size=0.4 0.3 0.1
Joints:
- removed joint base_to_caster
- removed joint base_to_left_wheel
- removed joint base_to_right_wheel
- added joint base_to_left_front_caster: type fixed, parent base_link, child left_front_caster, origin xyz=-0.15 0.15 -0.05 rpy=1.5708 0 0
- added joint base_to_left_rear_wheel: type continuous, parent base_link, child left_rear_wheel, origin xyz=0.15 0.15 -0.05 rpy=1.5708 0 0, axis 0 0 1
- added joint base_to_right_front_caster: type fixed, parent base_link, child right_front_caster, origin xyz=-0.15 -0.15 -0.05 rpy=1.5708 0 0
- added joint base_to_right_rear_wheel: type continuous, parent base_link, child right_rear_wheel, origin xyz=0.15 -0.15 -0.05 rpy=1.5708 0 0, axis 0 0 1

Commit message: corrected

File: src/mower_robot/urdf/mower_robot.urdf (robot description, URDF)
Before this commit: robot mower_robot, 6 links, 5 joints
Links:
- link base_link: mass 5.0 -> 2.0
- link left_front_caster: mass 0.5 -> 0.1
- link left_rear_wheel: mass 0.5 -> 0.2
- link lidar_link: mass 0.2 -> 0.1
- link right_front_caster: mass 0.5 -> 0.1
- link right_rear_wheel: mass 0.5 -> 0.2
Joints:
- joint base_to_lidar: origin xyz=0 0 0.1 -> xyz=0 0 0.1 rpy=0 0 0
